File: hardware/pcbs/AD7606/AD7606/AD7606.kicad_sch (KiCad schematic)
At the start: 27 parts, among them J2 H_16_2.54mm, SW1 SW_Reed_SPDT, SW2 SW_Reed_SPDT, SW3 SW_Reed_SPDT, SW4 SW_Reed_SPDT, U1 AD7606BSTZ

Commit message: Voltage supply of sEMG & ADC
Changed lines of the file:
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@@
 (kicad_sch
-	(version 20231120)
+	(version 20250114)
 	(generator "eeschema")
-	(generator_version "8.0")
+	(generator_version "9.0")
 	(paper "A4")
+	(text "3x0.1uF\n"
+		(exclude_from_sim no)
+		(at 147.32 40.132 0)
+		(effects
+			(font
+				(size 1.27 1.27)
+			)
+		)
+	)
 	(junction
 		(at 121.666 145.034)
@@
 		)
 	)
-	(text "3x0.1uF\n"
-		(exclude_from_sim no)
-		(at 147.32 40.132 0)
-		(effects
-			(font
-				(size 1.27 1.27)
-			)
-		)
-	)
 	(global_label "V5GND"
 		(shape input)
@@
 		)
 	)
+	(embedded_fonts no)
 )
