File: hardware/pcbs/ArmProthesis/sEMG_to_ADC_connector/sEMG_to_ADC_connector.kicad_pcb (KiCad board)
At the start: 2 copper layers, 54.1 x 38.9 mm, 13 parts, among them J1 Conn_01x01_Pin, J2 Conn_01x01_Pin, J3 Conn_01x01_Pin, J4 Conn_01x01_Pin, J5 Conn_01x01_Pin, J6 Conn_01x01_Pin, J7 Conn_01x01_Pin, J8 Conn_01x01_Pin, J9 Conn_01x08

Commit message: BMS v0.3 + main folder reconstruction
Parts:
- added G***: LOGO, LOGO, B.Cu at (132.1, 119.0)
- moved J1 0.50 mm to (152.0, 121.0)
- moved J2 0.50 mm to (152.0, 111.5)
- moved J7 0.50 mm to (113.0, 112.5)
- moved J8 0.50 mm to (113.0, 122.0)
- moved H2 0.25 mm to (110.0, 129.4)
- moved H3 0.25 mm to (155.2, 129.1)
