File: hardware/pcbs/BMS/BMS.kicad_sch (KiCad schematic)
At the start: 57 parts, among them J1 XT60-M, J2 XT60-F, J3 4-1971800-1, Q1 BSC014N04LSIATMA1, Q2 BSC014N04LSIATMA1, Q3 BSS84, SW1 CK_KMS2xxG, SW2 CK_KMS2xxG, SW3 CK_KMS2xxG, U1 BQ76920PW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

Commit message: BMS v0.2v + polishment of Vsupply  board
Parts:
- C1, C2: footprint Capacitor_SMD:C_0805_2012Metric_Pad1.18x1.45mm_HandSolder -> Capacitor_SMD:C_0603_1608Metric_Pad1.08x0.95mm_HandSolder; Website http://eu.mouser.com/ProductDetail/Murata-Electronics/GCJ21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 -> https://eu.mouser.com/ProductDetail/TDK/C1608X7R1H105K080AB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
- J1: footprint Connector_AMASS:AMASS_XT60-M_1x02_P7.20mm_Vertical -> Connector_AMASS:AMASS_XT60PW-M_1x02_P7.20mm_Horizontal
- J2: footprint Connector_AMASS:AMASS_XT60-F_1x02_P7.20mm_Vertical -> Connector_AMASS:AMASS_XT60PW-F_1x02_P7.20mm_Horizontal
- U3, U4: footprint Connector_JST:JST_GH_BM02B-GHS-TBT_1x02-1MP_P1.25mm_Vertical -> Connector_JST:JST_GH_SM02B-GHS-TB_1x02-1MP_P1.25mm_Horizontal
- renumbered D8 to D2, R28 to R17, R26 to R18, R29 to R19
Changed lines of the file:
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@@
 (kicad_sch
-	(version 20231120)
+	(version 20250114)
 	(generator "eeschema")
-	(generator_version "8.0")
+	(generator_version "9.0")
 	(paper "A4")
 	(junction
@@
 		(on_board yes)
 		(dnp no)
-		(property "Reference" "R26"
+		(property "Reference" "R18"
 			(at 20.828 176.022 0)
 			(effects
@@
 			)
 		)
-		(property "Footprint" "Capacitor_SMD:C_0805_2012Metric_Pad1.18x1.45mm_HandSolder"
+		(property "Footprint" "Capacitor_SMD:C_0603_1608Metric_Pad1.08x0.95mm_HandSolder"
 			(at 121.92 55.1688 0)
 			(effects
@@
 			)
 		)
-		(property "Website" "http://eu.mouser.com/ProductDetail/Murata-Electronics/GCJ21BR71H105MA01K?qs=QzBtWTOodeVZ%252BTk8SNChEw%3D%3D"
+		(property "Website" "https://eu.mouser.com/ProductDetail/TDK/C1608X7R1H105K080AB?qs=efUn273yAhdzCWVW9RXgig%3D%3D"
 			(at 118.11 56.134 0)
 			(effects
@@
 			)
 		)
-		(property "Footprint" "Connector_AMASS:AMASS_XT60-F_1x02_P7.20mm_Vertical"
+		(property "Footprint" "Connector_AMASS:AMASS_XT60PW-F_1x02_P7.20mm_Horizontal"
 			(at 259.588 89.154 0)
 			(effects
@@
 			)
 		)
-		(property "Footprint" "Connector_JST:JST_GH_BM02B-GHS-TBT_1x02-1MP_P1.25mm_Vertical"
+		(property "Footprint" "Connector_JST:JST_GH_SM02B-GHS-TB_1x02-1MP_P1.25mm_Horizontal"
 			(at 258.318 49.022 0)
 			(effects
@@
 			)
 		)
-		(property "Footprint" "Connector_AMASS:AMASS_XT60-M_1x02_P7.20mm_Vertical"
+		(property "Footprint" "Connector_AMASS:AMASS_XT60PW-M_1x02_P7.20mm_Horizontal"
 			(at 259.588 80.264 0)
 			(effects
@@
 			)
 		)
-		(property "Footprint" "Capacitor_SMD:C_0805_2012Metric_Pad1.18x1.45mm_HandSolder"
+		(property "Footprint" "Capacitor_SMD:C_0603_1608Metric_Pad1.08x0.95mm_HandSolder"
 			(at 106.172 86.1568 0)
 			(effects
@@
 			)
 		)
-		(property "Website" "http://eu.mouser.com/ProductDetail/Murata-Electronics/GCJ21BR71H105MA01K?qs=QzBtWTOodeVZ%252BTk8SNChEw%3D%3D"
+		(property "Website" "https://eu.mouser.com/ProductDetail/TDK/C1608X7R1H105K080AB?qs=efUn273yAhdzCWVW9RXgig%3D%3D"
 			(at 102.362 87.122 0)
 			(effects
@@
 		(on_board yes)
 		(dnp no)
-		(property "Reference" "D8"
+		(property "Reference" "D2"
 			(at 86.36 150.368 0)
 			(effects
@@
 		(on_board yes)
 		(dnp no)
-		(property "Reference" "R28"
+		(property "Reference" "R17"
 			(at 34.29 176.022 0)
 			(effects
@@
 		(on_board yes)
 		(dnp no)
-		(property "Reference" "R29"
+		(property "Reference" "R19"
 			(at 98.044 163.576 90)
 			(effects
@@
 			)
 		)
-		(property "Footprint" "Connector_JST:JST_GH_BM02B-GHS-TBT_1x02-1MP_P1.25mm_Vertical"
+		(property "Footprint" "Connector_JST:JST_GH_SM02B-GHS-TB_1x02-1MP_P1.25mm_Horizontal"
 			(at 258.318 57.658 0)
 			(effects
@@
 		)
 	)
+	(embedded_fonts no)
 )

Commit message: BMS v0.3 + main folder reconstruction
Parts:
- J3: footprint headers:XH_2.5mm -> Connector_JST:JST_XH_S4B-XH-A_1x04_P2.50mm_Horizontal
- U5: footprint Connector_PinHeader_2.54mm:PinHeader_2x05_P2.54mm_Vertical -> Connector_PinHeader_2.54mm:PinHeader_2x05_P2.54mm_Horizontal
Connections:
- net PA0: now also U5.8; no longer U5.3
- net PA1: now also U5.7; no longer U5.4
- net PA11: now also U5.4; no longer U5.7
- net PA12: now also U5.3; no longer U5.8
- net PA13: now also U5.6; no longer U5.5
- net PA14: now also U5.5; no longer U5.6
- net PA2: now also U5.10; no longer U5.1
- net PA3: now also U5.9; no longer U5.2
- net PA5: now also U5.1; no longer U5.10
- net PA6: now also U5.2; no longer U5.9
- net at C6.2, R3.2: now also J3.4; no longer J3.1
- net at C7.1, C8.2, R2.2: now also J3.3; no longer J3.2
- net at C8.1, C9.2, R4.2: now also J3.2; no longer J3.3
- net at C9.1, R5.2: now also J3.1; no longer J3.4
