File: hardware/pcbs/ArmProthesis/BMS.kicad_sch (KiCad schematic)
At the start: 49 parts, among them J1 XT60-M, J2 XT60-F, J4 Conn_01x03, Q1 BSC014N04LSIATMA1, Q2 BSC014N04LSIATMA1, SW1 CK_KMS2xxG, SW2 CK_KMS2xxG, SW4 CK_KMS2xxG, U2 BQ76905RGRR, U6 STM32C011F6Px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

Commit message: BMS board fixes
Parts:
- added D4: 1N4148WT, Diode_SMD:D_SOD-523, symbol Diode:1N4148WT
- added R13: 100, Resistor_SMD:R_0402_1005Metric, symbol Device:R
- C10: value 4.7pF -> 10uF
Connections:
- net PACK+: now also D4.2 (A)
- net at C1.2, U2.16 (REGSRC): now also R13.1; no longer R5.1, U2.18 (VC5)
- net BMS_GND renamed PACK-
- new net: D4.1 (K), R13.2
- new net: R5.1, U2.18 (VC5)
Other:
- moved on the sheet: C10, H1, H2, H3, H4, J1, J2, U3, U4

Commit message: Ordered versions
Parts:
- removed SW1, SW2, SW4: CK_KMS2xxG, Button_Switch_SMD:SW_SPST_CK_KMS2xxG, symbol Switch:CK_KMS2xxG
- added SW1, SW2, SW3: SW_Push, Button_Switch_SMD:SW_SPST_B3U-3000P, symbol Switch:SW_Push
- C10: value 10uF -> 1uF; LCSC C167420 -> C14445
- C11: LCSC C2918502 -> C105197
- J1: LCSC (none) -> C98732
- J2: LCSC (none) -> C428722
- J4: footprint Connector_JST:JST_GH_BM03B-GHS-TBT_1x03-1MP_P1.25mm_Vertical -> Connector_JST:JST_GH_SM03B-GHS-TB_1x03-1MP_P1.25mm_Horizontal; LCSC (none) -> C514175
- R11: LCSC C60490 -> C93945
- R4: LCSC C60490 -> C25741
- U2: LCSC (none) -> C22394458
- U3, U4: value ~ -> JST-GH
- U5: value ~ -> PIN-HEADER; LCSC (none) -> C492433
- Y1: value Crystal -> YXC X321532768KGD2SI; LCSC C519280 -> C620155
Connections:
- net +3.3V: now also SW3.1
- net GND: now also SW2.1
- net PWROFF: now also SW3.2
- net at U6.6 (PF2): now also SW2.2
- net at R2.1, U2.1 (VC3A), U2.19 (VC4A)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: now also SW1.2
- net at C6.2, R3.2: now also J4.3 (Pin_3); no longer J4.1 (Pin_1)
- net at C9.1, R5.2: now also J4.1 (Pin_1); no longer J4.3 (Pin_3)
- net at D1.2 (A): now also SW1.1
Other:
- moved on the sheet: R12
