File: hardware/pcbs/ArmProthesis/ArmProthesis.kicad_sch (KiCad schematic)
At the start: 0 parts

Commit message: Synced the files with the latest versions
The files that were merged were one version behind. Also the names of the projects were renamed for clarity.
Parts:
- added U2, U3: ~, symbol Drawings:arrow
Connections:
- new net: U2., U3.
Other:
- note added: "+8.4V"
- note added: "EXACT ANGLE CONTROL CURRENT ANGLE FEEDBACK The motors aren't chosen yet. They are to be added to the system in the future."
- note added: "PARALLEL MODE"
- note added: "SCL SDA ALERT POWEROFF"
