File: hardware/pcbs/ArmProthesis/BMS.kicad_pcb (KiCad board)
At the start: 4 copper layers, 64.1 x 55.2 mm, 49 parts, among them J1 XT60-M, J2 XT60-F, J4 Conn_01x03, Q1 BSC014N04LSIATMA1, Q2 BSC014N04LSIATMA1, SW1 CK_KMS2xxG, SW2 CK_KMS2xxG, SW4 CK_KMS2xxG, U2 BQ76905RGRR, U6 STM32C011F6Px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

Commit message: Ordered versions
Parts:
- removed SW4: CK_KMS2xxG, Button_Switch_SMD:SW_SPST_CK_KMS2xxG
- added D4: 1N4148WT, Diode_SMD:D_SOD-523, F.Cu at (151.9, 101.1)
- added R13: 100, Resistor_SMD:R_0402_1005Metric, F.Cu at (151.9, 98.7)
- added SW3: SW_Push, Button_Switch_SMD:SW_SPST_B3U-3000P, F.Cu at (164.1, 117.6)
- C10: value 4.7pF -> 1uF
- J4: footprint Connector_JST:JST_GH_BM03B-GHS-TBT_1x03-1MP_P1.25mm_Vertical -> Connector_JST:JST_GH_SM03B-GHS-TB_1x03-1MP_P1.25mm_Horizontal
- SW1, SW2: value CK_KMS2xxG -> SW_Push; footprint Button_Switch_SMD:SW_SPST_CK_KMS2xxG -> Button_Switch_SMD:SW_SPST_B3U-3000P
- U3, U4: value ~ -> JST-GH
- U5: value ~ -> PIN-HEADER
- Y1: value Crystal -> YXC X321532768KGD2SI
- moved R12 2.51 mm to (165.2, 120.1), turned to 180 degrees
- moved C11 1.74 mm to (155.6, 99.0)
- moved R8 1.74 mm to (155.0, 101.4)
- moved D3 1.73 mm to (154.8, 103.0)
- moved SW1 1.66 mm to (140.1, 93.8)
- moved D1 1.54 mm to (143.1, 94.8)
- moved R11 1.54 mm to (143.1, 91.8)
- moved R4 1.54 mm to (144.9, 91.8)
- moved SW2 1.43 mm to (141.6, 118.3)
- moved J2 0.26 mm to (130.0, 88.9)
- turned J4 to 90 degrees
Connections:
- net /BMS_GND renamed /PACK-
- net PACK+ renamed /PACK+
- C1 pad 1: PACK- -> GND
- C10 pad 1: PACK- -> GND
- C11 pad 1: PACK- -> GND
- C12 pad 2: PACK- -> GND
- C13 pad 2: PACK- -> GND
- C14 pad 2: PACK- -> GND
- C3 pad 1: PACK- -> GND
- C4 pad 1: PACK- -> GND
- C6 pad 1: PACK- -> GND
- C6 pad 2: Net-(J4-Pin_1) -> Net-(J4-Pin_3)
- C7 pad 2: PACK- -> GND
- C9 pad 1: Net-(J4-Pin_3) -> Net-(J4-Pin_1)
- J1 pad 1: PACK- -> GND
- R1 pad 2: PACK- -> GND
- R12 pad 2: PACK- -> GND
- R3 pad 2: Net-(J4-Pin_1) -> Net-(J4-Pin_3)
- R4 pad 2: PACK- -> GND
- R5 pad 1: Net-(U2-REGSRC) -> Net-(U2-VC5)
- R5 pad 2: Net-(J4-Pin_3) -> Net-(J4-Pin_1)
- R7 pad 1: PACK- -> GND
- SW1 pad 1: Net-(U2-VC1) -> Net-(D1-A)
- SW1 pad 2: Net-(D1-A) -> Net-(U2-VC1)
- SW2 pad 1: Net-(U6-PF2) -> GND
- SW2 pad 2: PACK- -> Net-(U6-PF2)
- U2 pad 11: PACK- -> GND
- U2 pad 18: Net-(U2-REGSRC) -> Net-(U2-VC5)
- U2 pad 21: PACK- -> GND
- U6 pad 5: PACK- -> GND
Routing:
- net PACK-: track 29.7 -> 0.00 mm, vias 29 -> 0
- net GND: track 0.00 -> 23.3 mm, vias 0 -> 26
- net Net-(U2-VC1): track 29.2 -> 19.1 mm
- net Net-(U2-REGSRC): track 7.69 -> 0.80 mm, vias 2 -> 0
- net +3.3V: track 54.3 -> 49.5 mm
- net Net-(D1-A): track 6.44 -> 3.06 mm
- net /PACK-: track 17.3 -> 14.3 mm
- net Net-(U2-VC5): track 0.00 -> 2.73 mm
- net /PACK+: track 6.92 -> 8.95 mm
- net Net-(U6-PF2): track 8.88 -> 6.98 mm
- net Net-(U2-TS): track 14.7 -> 13.1 mm
- net Net-(D4-K): track 0.00 -> 1.11 mm
- net PWROFF: track 15.8 -> 15.0 mm
- net Net-(J4-Pin_3): track 25.2 -> 24.4 mm
- net Net-(J4-Pin_1): track 24.4 -> 25.1 mm
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- added copper zone on In1.Cu, net GND
- removed copper zone on In1.Cu, net PACK-
Other:
- board text added: "BMS v0.8"
- board text removed: "BMS v0.7"
