File: hardware/pcbs/ArmProthesis/EMG sensors.kicad_sch (KiCad schematic)
At the start: 29 parts, among them J1 Conn_01x02_Pin, J2 DNP, J3 Conn_01x03_Pin, U1 DNP, U2 DNP, U3 LME49726MY, U4 INA326, U5 LME49726MY

Commit message: Synced the files with the latest versions
The files that were merged were one version behind. Also the names of the projects were renamed for clarity.
Other:
- note added: "2x4mm ECG electrode snaps"
- note added: "DIN 1.5mm for third electrode to bone"
Changed lines of the file:
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@@
+		)
+	)
+	(text "DIN 1.5mm\nfor third electrode\nto bone"
+		(exclude_from_sim no)
+		(at 144.272 30.734 0)
+		(effects
+			(font
+				(size 1.27 1.27)
+			)
+		)
+	)
+	(text "2x4mm ECG \nelectrode snaps"
+		(exclude_from_sim no)
+		(at 178.816 29.972 0)
+		(effects
+			(font
+				(size 1.27 1.27)
+			)
 		)
 	)
